File: jfmicro/testpcb/testpcb.sch (KiCad schematic (older format))
At the start: 32 parts, among them J1 Type C, K1 KEYSW, K2 KEYSW, K3 KEYSW, K4 KEYSW, K5 KEYSW, K6 KEYSW, SW1 SW_PUSH, SW2 Rotary_Encoder_Switch, U1 ATMEGA32U4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

Commit message: micro revision two and more comps
Parts:
- J1: footprint Type-C:HRO-TYPE-C-31-M-12-Assembly -> Type-C:12401598E4#2A
- R1, R2, R3, R4, R5, R6: footprint Resistor_SMD:R_1210_3225Metric -> Resistor_SMD:R_0805_2012Metric
Changed lines of the file:
@@
 F 0 "R2" V 4900 2750 50  0000 C CNN
 F 1 "10k" V 4950 2950 50  0000 C CNN
-F 2 "Resistor_SMD:R_1210_3225Metric" V 4880 2950 50  0001 C CNN
+F 2 "Resistor_SMD:R_0805_2012Metric" V 4880 2950 50  0001 C CNN
 F 3 "~" H 4950 2950 50  0001 C CNN
 	1    4950 2950
@@
 F 0 "J1" H 850 2500 60  0000 C CNN
 F 1 "Type C" V 500 1900 60  0000 C CNN
-F 2 "Type-C:HRO-TYPE-C-31-M-12-Assembly" H 1050 1850 60  0001 C CNN
+F 2 "Type-C:12401598E4#2A" H 1050 1850 60  0001 C CNN
 F 3 "" H 1050 1850 60  0001 C CNN
 	1    1050 1850
@@
 F 0 "R1" V 1450 2800 50  0000 C CNN
 F 1 "10k" V 1550 2800 50  0000 C CNN
-F 2 "Resistor_SMD:R_1210_3225Metric" V 1480 2800 50  0001 C CNN
+F 2 "Resistor_SMD:R_0805_2012Metric" V 1480 2800 50  0001 C CNN
 F 3 "~" H 1550 2800 50  0001 C CNN
 	1    1550 2800
@@
 F 0 "R3" V 1450 1600 50  0000 C CNN
 F 1 "5.1k" V 1550 1600 50  0000 C CNN
-F 2 "Resistor_SMD:R_1210_3225Metric" V 1480 1600 50  0001 C CNN
+F 2 "Resistor_SMD:R_0805_2012Metric" V 1480 1600 50  0001 C CNN
 F 3 "~" H 1550 1600 50  0001 C CNN
 	1    1550 1600
@@
 F 0 "R4" V 1450 2200 50  0000 C CNN
 F 1 "5.1k" V 1550 2200 50  0000 C CNN
-F 2 "Resistor_SMD:R_1210_3225Metric" V 1480 2200 50  0001 C CNN
+F 2 "Resistor_SMD:R_0805_2012Metric" V 1480 2200 50  0001 C CNN
 F 3 "~" H 1550 2200 50  0001 C CNN
 	1    1550 2200
@@
 F 0 "R5" V 2200 2200 50  0000 C CNN
 F 1 "22p" V 2250 2050 50  0000 C CNN
-F 2 "Resistor_SMD:R_1210_3225Metric" V 2180 2050 50  0001 C CNN
+F 2 "Resistor_SMD:R_0805_2012Metric" V 2180 2050 50  0001 C CNN
 F 3 "~" H 2250 2050 50  0001 C CNN
 	1    2250 2050
@@
 F 0 "R6" V 2200 2300 50  0000 C CNN
 F 1 "22p" V 2250 2150 50  0000 C CNN
-F 2 "Resistor_SMD:R_1210_3225Metric" V 2180 2150 50  0001 C CNN
+F 2 "Resistor_SMD:R_0805_2012Metric" V 2180 2150 50  0001 C CNN
 F 3 "~" H 2250 2150 50  0001 C CNN
 	1    2250 2150
